File: hardware/espduino-01/espduino-01.sch (EAGLE design)
At the start: 20 parts, among them U1 FT231XS

Commit message: Rev 2 of espduino-m2
Parts:
- added U$2, U$3: MOUNTING-HOLEM1.6, jumper-parts:MOUNTING-HOLEM1.6
Connections:
- net GND: now also U$2.GND, U$3.GND
Changed lines of the file:
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@@
 <?xml version="1.0" encoding="utf-8"?>
 <!DOCTYPE eagle SYSTEM "eagle.dtd">
-<eagle version="7.1.0">
+<eagle version="7.2.0">
 <drawing>
 <settings>
@@
 <part name="C2" library="resistor" deviceset="C-US" device="C0603" value="10uF"/>
 <part name="U2" library="jumper-parts" deviceset="USB-AB" device=""/>
+<part name="U$2" library="jumper-parts" deviceset="MOUNTING-HOLE" device="M1.6"/>
+<part name="U$3" library="jumper-parts" deviceset="MOUNTING-HOLE" device="M1.6"/>
+<part name="GND10" library="SparkFun-Aesthetics" deviceset="GND" device=""/>
+<part name="GND12" library="SparkFun-Aesthetics" deviceset="GND" device=""/>
 </parts>
 <sheets>
@@
 <instance part="C2" gate="G$1" x="48.26" y="15.24"/>
 <instance part="U2" gate="G$1" x="20.32" y="58.42" rot="R180"/>
+<instance part="U$2" gate="G$1" x="-2.54" y="76.2"/>
+<instance part="U$3" gate="G$1" x="-2.54" y="63.5"/>
+<instance part="GND10" gate="1" x="-5.08" y="66.04" rot="R270"/>
+<instance part="GND12" gate="1" x="-5.08" y="78.74" rot="R270"/>
 </instances>
 <busses>
@@
 <pinref part="GND8" gate="1" pin="GND"/>
 </segment>
-</net>
+<segment>
+<pinref part="U$3" gate="G$1" pin="GND"/>
+<pinref part="GND10" gate="1" pin="GND"/>
+</segment>
+<segment>
+<pinref part="U$2" gate="G$1" pin="GND"/>
+<pinref part="GND12" gate="1" pin="GND"/>
+</segment>
+</net>
