File: hardware/espduino-12/espduino-12.sch (EAGLE design)
At the start: 18 parts, among them U1 FT231XS

Commit message: Rev 2 of espduino-m2
Parts:
- added SJ1: (no value), jumper-parts:SJCUTTABLE
- C1: value 4.7uF -> 10uF
- R3, R4, R5: value 10k -> 4.7k
Connections:
- new net VUSB: SJ1.1, U2.VBUS
- net 5V: now also SJ1.2; no longer U2.VBUS
Changed lines of the file:
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@@
 <?xml version="1.0" encoding="utf-8"?>
 <!DOCTYPE eagle SYSTEM "eagle.dtd">
-<eagle version="7.1.0">
+<eagle version="7.2.0">
 <drawing>
 <settings>
@@
 <part name="GND5" library="SparkFun-Aesthetics" deviceset="GND" device=""/>
 <part name="GND7" library="SparkFun-Aesthetics" deviceset="GND" device=""/>
-<part name="C1" library="resistor" deviceset="C-US" device="C0603" value="4.7uF"/>
-<part name="R3" library="resistor" deviceset="R-US_" device="R0603" value="10k"/>
-<part name="R4" library="resistor" deviceset="R-US_" device="R0603" value="10k"/>
-<part name="R5" library="resistor" deviceset="R-US_" device="R0603" value="10k"/>
+<part name="C1" library="resistor" deviceset="C-US" device="C0603" value="10uF"/>
+<part name="R3" library="resistor" deviceset="R-US_" device="R0603" value="4.7k"/>
+<part name="R4" library="resistor" deviceset="R-US_" device="R0603" value="4.7k"/>
+<part name="R5" library="resistor" deviceset="R-US_" device="R0603" value="4.7k"/>
 <part name="SUPPLY1" library="SparkFun-Aesthetics" deviceset="3.3V" device=""/>
 <part name="SUPPLY2" library="SparkFun-Aesthetics" deviceset="3.3V" device=""/>
@@
 <part name="SUPPLY14" library="SparkFun-Aesthetics" deviceset="3.3V" device=""/>
 <part name="SUPPLY15" library="SparkFun-Aesthetics" deviceset="3.3V" device=""/>
+<part name="SJ1" library="jumper-parts" deviceset="SJ" device="CUTTABLE"/>
 </parts>
 <sheets>
@@
 <instance part="C7" gate="G$1" x="10.16" y="20.32"/>
 <instance part="C8" gate="G$1" x="30.48" y="20.32"/>
-<instance part="SUPPLY9" gate="G$1" x="33.02" y="81.28"/>
+<instance part="SUPPLY9" gate="G$1" x="0" y="81.28" rot="R270"/>
 <instance part="SUPPLY10" gate="G$1" x="63.5" y="76.2"/>
 <instance part="SUPPLY12" gate="G$1" x="83.82" y="93.98"/>
@@
 <instance part="SUPPLY14" gate="G$1" x="58.42" y="-35.56" rot="R90"/>
 <instance part="SUPPLY15" gate="G$1" x="78.74" y="-48.26" rot="R90"/>
+<instance part="SJ1" gate="1" x="-5.08" y="81.28"/>
 </instances>
 <busses>
@@
 </segment>
 <segment>
-<wire x1="25.4" y1="63.5" x2="33.02" y2="63.5" width="0.1524" layer="91"/>
-<wire x1="33.02" y1="63.5" x2="33.02" y2="81.28" width="0.1524" layer="91"/>
-<pinref part="SUPPLY9" gate="G$1" pin="5V"/>
-<pinref part="U2" gate="G$1" pin="VBUS"/>
-</segment>
-<segment>
 <pinref part="U1" gate="G$1" pin="VCC"/>
 <wire x1="66.04" y1="71.12" x2="63.5" y2="71.12" width="0.1524" layer="91"/>
@@
 <wire x1="83.82" y1="91.44" x2="83.82" y2="93.98" width="0.1524" layer="91"/>
 <pinref part="SUPPLY12" gate="G$1" pin="5V"/>
+</segment>
+<segment>
+<pinref part="SJ1" gate="1" pin="2"/>
+<pinref part="SUPPLY9" gate="G$1" pin="5V"/>
 </segment>
 </net>
@@
 </segment>
 </net>
+<net name="VUSB" class="1">
+<segment>
+<wire x1="25.4" y1="63.5" x2="33.02" y2="63.5" width="0.1524" layer="91"/>
+<pinref part="U2" gate="G$1" pin="VBUS"/>
+<label x="33.02" y="63.5" size="1.778" layer="95" xref="yes"/>
+</segment>
+<segment>
+<pinref part="SJ1" gate="1" pin="1"/>
+<wire x1="-10.16" y1="81.28" x2="-15.24" y2="81.28" width="0.1524" layer="91"/>
+<label x="-15.24" y="81.28" size="1.778" layer="95" rot="R180" xref="yes"/>
+</segment>
+</net>
